File: BPS/Master-Nucleo/BPS-Nucleo.sch (KiCad schematic (older format))
At the start: 14 parts, among them J12 Conn_01x04, U1 NUCLEO144-F412ZG

Commit message: Connected all PCB components. Space in middle cannot be utilized. Distance between traces and copper must be less than .127mm or 5 mils according to manufacturer capabilities.
Parts:
- U1: symbol utsvt-bps:NUCLEO144-F412ZG -> BPS-Nucleo-rescue:NUCLEO144-F412ZG-utsvt-bps
Changed lines of the file:
@@
 EESchema Schematic File Version 4
 LIBS:BPS-Nucleo-cache
-EELAYER 26 0
+EELAYER 30 0
 EELAYER END
 $Descr A3 16535 11693
@@
 $EndDescr
 $Comp
-L utsvt-bps:NUCLEO144-F412ZG U1
+L BPS-Nucleo-rescue:NUCLEO144-F412ZG-utsvt-bps U1
 U 1 1 5D3D798F
 P 8200 5650
