File: BPS/Master-Nucleo/CAN.sch (KiCad schematic (older format))
At the start: 23 parts, among them J11 CAN_Out, U14 ADM3055E, U5 CDSOT23-T24CAN

Commit message: Connected all PCB components. Space in middle cannot be utilized. Distance between traces and copper must be less than .127mm or 5 mils according to manufacturer capabilities.
Parts:
- J11: symbol utsvt-connectors:CANConnector -> BPS-Nucleo-rescue:CANConnector-utsvt-connectors
- U14: symbol utsvt-chips:ADM3055E -> BPS-Nucleo-rescue:ADM3055E-utsvt-chips
- U5: symbol utsvt-chips:CDSOT23-T24CAN -> BPS-Nucleo-rescue:CDSOT23-T24CAN-utsvt-chips
Changed lines of the file:
@@
 EESchema Schematic File Version 4
 LIBS:BPS-Nucleo-cache
-EELAYER 26 0
+EELAYER 30 0
 EELAYER END
 $Descr A4 11693 8268
@@
 $EndDescr
 $Comp
-L utsvt-connectors:CANConnector J11
+L BPS-Nucleo-rescue:CANConnector-utsvt-connectors J11
 U 1 1 5C2B42F3
 P 9250 3800
@@
 $EndComp
 $Comp
-L utsvt-chips:ADM3055E U14
+L BPS-Nucleo-rescue:ADM3055E-utsvt-chips U14
 U 1 1 5C2B4359
 P 4350 3600
@@
 $EndComp
 $Comp
-L utsvt-chips:CDSOT23-T24CAN U5
+L BPS-Nucleo-rescue:CDSOT23-T24CAN-utsvt-chips U5
 U 1 1 5C2B43A0
 P 8100 2850
