File: BPS/Master-Nucleo/Contactor.sch (KiCad schematic (older format))
At the start: 20 parts, among them J1 ContactorConnector, Q1 VND5N07-E, Q2 NTR4003NT1G, U2 BAS70-04, U3 SI8261ABC-IS

Commit message: Connected all PCB components. Space in middle cannot be utilized. Distance between traces and copper must be less than .127mm or 5 mils according to manufacturer capabilities.
Parts:
- U2: symbol utsvt-bps:BAS70-04 -> BPS-Nucleo-rescue:BAS70-04-utsvt-bps
- U3: symbol utsvt-bps:SI8261ABC-IS -> BPS-Nucleo-rescue:SI8261ABC-IS-utsvt-bps
Changed lines of the file:
@@
 EESchema Schematic File Version 4
 LIBS:BPS-Nucleo-cache
-EELAYER 26 0
+EELAYER 30 0
 EELAYER END
 $Descr A4 11693 8268
@@
 	8700 4200 8700 4100
 $Comp
-L utsvt-bps:BAS70-04 U2
+L BPS-Nucleo-rescue:BAS70-04-utsvt-bps U2
 U 1 1 5C304528
 P 8200 3500
+AR Path="/5C304528" Ref="U2"  Part="1"
+AR Path="/5D3DB608/5C304528" Ref="U2"  Part="1"
 F 0 "U2" H 8072 3346 50  0000 R CNN
 F 1 "BAS70-04" H 8072 3255 50  0000 R CNN
@@
 Connection ~ 5200 3850
 $Comp
-L utsvt-bps:SI8261ABC-IS U3
+L BPS-Nucleo-rescue:SI8261ABC-IS-utsvt-bps U3
 U 1 1 5C30F57F
 P 3750 3550
