File: BPS/Master-Nucleo/I2C.sch (KiCad schematic (older format))
At the start: 5 parts, among them J3 Conn_01x03, U6 M24128

Commit message: Connected all PCB components. Space in middle cannot be utilized. Distance between traces and copper must be less than .127mm or 5 mils according to manufacturer capabilities.
Parts:
- U6: symbol utsvt-bps:M24128 -> BPS-Nucleo-rescue:M24128-utsvt-bps
Changed lines of the file:
@@
 EESchema Schematic File Version 4
 LIBS:BPS-Nucleo-cache
-EELAYER 26 0
+EELAYER 30 0
 EELAYER END
 $Descr A4 11693 8268
 encoding utf-8
-Sheet 5 7
+Sheet 4 7
 Title ""
 Date ""
@@
 GND
 $Comp
-L utsvt-bps:M24128 U6
+L BPS-Nucleo-rescue:M24128-utsvt-bps U6
 U 1 1 5C3511BE
 P 4250 2800
