File: BPS/Master-Nucleo/Misc.sch (KiCad schematic (older format))
At the start: 34 parts, among them J4 FrontFans, J5 ErrorLightConnector, J6 BackFans, Q3 NTR4003NT1G, Q4 NTR4003NT1G, U7 SI8261ABC-IS

Commit message: Connected all PCB components. Space in middle cannot be utilized. Distance between traces and copper must be less than .127mm or 5 mils according to manufacturer capabilities.
Parts:
- U7: symbol utsvt-bps:SI8261ABC-IS -> BPS-Nucleo-rescue:SI8261ABC-IS-utsvt-bps
Changed lines of the file:
@@
 EESchema Schematic File Version 4
 LIBS:BPS-Nucleo-cache
-EELAYER 26 0
+EELAYER 30 0
 EELAYER END
 $Descr A4 11693 8268
@@
 Error Light
 $Comp
-L utsvt-bps:SI8261ABC-IS U7
+L BPS-Nucleo-rescue:SI8261ABC-IS-utsvt-bps U7
 U 1 1 5C35EBB6
 P 3350 3150
