File: BPS/Master-Nucleo/PowerDist.sch (KiCad schematic (older format))
At the start: 11 parts, among them J2 CarPowerConnector, U4 RI3-1205S

Commit message: Connected all PCB components. Space in middle cannot be utilized. Distance between traces and copper must be less than .127mm or 5 mils according to manufacturer capabilities.
Parts:
- J2: symbol utsvt-connectors:CarPowerConnector -> BPS-Nucleo-rescue:CarPowerConnector-utsvt-connectors
- L1: symbol utsvt-bps:SRF0905-100Y -> BPS-Nucleo-rescue:SRF0905-100Y-utsvt-bps
- U4: symbol utsvt-power-regulators:RI3-1205S -> BPS-Nucleo-rescue:RI3-1205S-utsvt-power-regulators
Changed lines of the file:
@@
 EESchema Schematic File Version 4
 LIBS:BPS-Nucleo-cache
-EELAYER 26 0
+EELAYER 30 0
 EELAYER END
 $Descr A4 11693 8268
@@
 $EndDescr
 $Comp
-L utsvt-connectors:CarPowerConnector J2
+L BPS-Nucleo-rescue:CarPowerConnector-utsvt-connectors J2
 U 1 1 5C35F236
 P 2100 3400
@@
 	4000 2750 4000 2850
 $Comp
-L utsvt-power-regulators:RI3-1205S U4
+L BPS-Nucleo-rescue:RI3-1205S-utsvt-power-regulators U4
 U 1 1 5C38C4FE
 P 4550 3200
@@
 	2700 3600 4000 3600
 $Comp
-L utsvt-bps:SRF0905-100Y L1
+L BPS-Nucleo-rescue:SRF0905-100Y-utsvt-bps L1
 U 1 1 5C35FFD4
 P 2950 3150
